Commit message: replace inf property with builtin global

File: bmb_description/urdf/aris.urdf.xacro (robot description, xacro)
@@ -1,5 +1,4 @@
 <?xml version="1.0"?>
 <robot xmlns:xacro="http://www.ros.org/wiki/xacro" name="aris">
-    <xacro:property name="inf" value="1000000000" />
     <link name="body">
         <visual>
@@ -49,5 +48,5 @@
         <origin xyz="-1.45 3.7 1.5" rpy="0.05 0 -0.12"/>
         <axis xyz="0 1 0"/>
-        <limit lower="${radians(-30)}" upper="${radians(30)}" velocity="${inf}" effort="${inf}"/>
+        <limit lower="${radians(-30)}" upper="${radians(30)}" velocity="inf" effort="inf"/>
     </joint>
     <!-- Right Aileron -->
@@ -65,5 +64,5 @@
         <origin xyz="0 0 0" rpy="0 0 0"/>
         <axis xyz="0 1 0"/>
-        <limit lower="${radians(-30)}" upper="${radians(30)}" velocity="${inf}" effort="${inf}"/>
+        <limit lower="${radians(-30)}" upper="${radians(30)}" velocity="inf" effort="inf"/>
     </joint>
     <!-- Elevator -->
@@ -81,5 +80,5 @@
         <origin xyz="0 0 0" rpy="0 0 0"/>
         <axis xyz="0 1 0"/>
-        <limit lower="${radians(-30)}" upper="${radians(30)}" velocity="${inf}" effort="${inf}"/>
+        <limit lower="${radians(-30)}" upper="${radians(30)}" velocity="inf" effort="inf"/>
     </joint>
     <gazebo>

Commit message: fix bugs in urdf

File: bmb_description/urdf/aris.urdf.xacro (robot description, xacro)
@@ -1,4 +1,5 @@
 <?xml version="1.0"?>
 <robot xmlns:xacro="http://www.ros.org/wiki/xacro" name="aris">
+    <xacro:property name="infty" value="${1e9}"/>
     <link name="body">
         <visual>
@@ -8,5 +9,5 @@
         </visual>
         <inertial>
-            <mass>3.068</mass>
+            <mass value="3.068"/>
             <inertia ixx="12.327" ixy="-3.07" ixz="0.739"
                      iyy="1.711" iyz="-2.789" izz="12.659"/>
@@ -45,8 +46,8 @@
     <joint name="body_to_left_aileron" type="revolute">
         <parent link="body"/>
-        <child link="body_to_left_aileron"/>
+        <child link="left_aileron"/>
         <origin xyz="-1.45 3.7 1.5" rpy="0.05 0 -0.12"/>
         <axis xyz="0 1 0"/>
-        <limit lower="${radians(-30)}" upper="${radians(30)}" velocity="inf" effort="inf"/>
+        <limit lower="${radians(-30)}" upper="${radians(30)}" velocity="${infty}" effort="${infty}"/>
     </joint>
     <!-- Right Aileron -->
@@ -61,8 +62,8 @@
     <joint name="body_to_right_aileron" type="revolute">
         <parent link="body"/>
-        <child link="body_to_right_aileron"/>
+        <child link="right_aileron"/>
         <origin xyz="0 0 0" rpy="0 0 0"/>
         <axis xyz="0 1 0"/>
-        <limit lower="${radians(-30)}" upper="${radians(30)}" velocity="inf" effort="inf"/>
+        <limit lower="${radians(-30)}" upper="${radians(30)}" velocity="${infty}" effort="${infty}"/>
     </joint>
     <!-- Elevator -->
@@ -77,8 +78,8 @@
     <joint name="body_to_elevator" type="revolute">
         <parent link="body"/>
-        <child link="body_to_elevator"/>
+        <child link="elevator"/>
         <origin xyz="0 0 0" rpy="0 0 0"/>
         <axis xyz="0 1 0"/>
-        <limit lower="${radians(-30)}" upper="${radians(30)}" velocity="inf" effort="inf"/>
+        <limit lower="${radians(-30)}" upper="${radians(30)}" velocity="${infty}" effort="${infty}"/>
     </joint>
     <gazebo>

Commit message: scale meshes from mm to m

File: bmb_description/urdf/aris.urdf.xacro (robot description, xacro)
@@ -5,5 +5,7 @@
         <visual>
             <geometry>
-                <mesh filename="package://bmb_description/meshes/body.stl"/>
+                <!-- All meshes are in mm -->
+                <mesh filename="package://bmb_description/meshes/body.stl"
+                      scale="0.001 0.001 0.001"/>
             </geometry>
         </visual>
@@ -27,5 +29,6 @@
         <visual>
             <geometry>
-                <mesh filename="package://bmb_description/meshes/propeller.stl"/>
+                <mesh filename="package://bmb_description/meshes/propeller.stl"
+                      scale="0.001 0.001 0.001"/>
             </geometry>
         </visual>
@@ -43,5 +46,6 @@
         <visual>
             <geometry>
-                <mesh filename="package://bmb_description/meshes/left_aileron.stl"/>
+                <mesh filename="package://bmb_description/meshes/left_aileron.stl"
+                      scale="0.001 0.001 0.001"/>
             </geometry>
         </visual>
@@ -59,5 +63,6 @@
         <visual>
             <geometry>
-                <mesh filename="package://bmb_description/meshes/right_aileron.stl"/>
+                <mesh filename="package://bmb_description/meshes/right_aileron.stl"
+                      scale="0.001 0.001 0.001"/>
             </geometry>
         </visual>
@@ -75,5 +80,6 @@
         <visual>
             <geometry>
-                <mesh filename="package://bmb_description/meshes/elevator.stl"/>
+                <mesh filename="package://bmb_description/meshes/elevator.stl"
+                      scale="0.001 0.001 0.001"/>
             </geometry>
         </visual>

Commit message: resize collision box

File: bmb_description/urdf/aris.urdf.xacro (robot description, xacro)
@@ -17,5 +17,5 @@
         <collision>
             <geometry>
-                <box size="1 2 0.5"/>
+                <box size="1.5 2.1 0.4"/>
             </geometry>
         </collision>

Commit message: correct left aileron origins

File: bmb_description/urdf/aris.urdf.xacro (robot description, xacro)
@@ -50,10 +50,10 @@
             </geometry>
         </visual>
-        <origin xyz="0 0 0" rpy="0 0 0"/>
+        <origin xyz="-1.45 3.7 1.5" rpy="0.05 0 -0.12"/>
     </link>
     <joint name="body_to_left_aileron" type="revolute">
         <parent link="body"/>
         <child link="left_aileron"/>
-        <origin xyz="-1.45 3.7 1.5" rpy="0.05 0 -0.12"/>
+        <origin xyz="0 0 0" rpy="0 0 0"/>
         <axis xyz="0 1 0"/>
         <limit lower="${radians(-30)}" upper="${radians(30)}" velocity="${infty}" effort="${infty}"/>

Commit message: update joint locations

File: bmb_description/urdf/aris.urdf.xacro (robot description, xacro)
@@ -38,5 +38,5 @@
         <parent link="body"/>
         <child link="propeller"/>
-        <origin xyz="0 0 0" rpy="0 0 0"/>
+        <origin xyz="0.4244 0 0.1638" rpy="0 0 0"/>
         <axis xyz="1 0 0"/>
     </joint>
@@ -55,5 +55,5 @@
         <parent link="body"/>
         <child link="left_aileron"/>
-        <origin xyz="0 0 0" rpy="0 0 0"/>
+        <origin xyz="-0.2649 0 0.1714" rpy="0 0 0"/>
         <axis xyz="0 1 0"/>
         <limit lower="${radians(-30)}" upper="${radians(30)}" velocity="${infty}" effort="${infty}"/>
@@ -72,5 +72,5 @@
         <parent link="body"/>
         <child link="right_aileron"/>
-        <origin xyz="0 0 0" rpy="0 0 0"/>
+        <origin xyz="-0.2649 0 0.1714" rpy="0 0 0"/>
         <axis xyz="0 1 0"/>
         <limit lower="${radians(-30)}" upper="${radians(30)}" velocity="${infty}" effort="${infty}"/>
@@ -89,5 +89,5 @@
         <parent link="body"/>
         <child link="elevator"/>
-        <origin xyz="0 0 0" rpy="0 0 0"/>
+        <origin xyz="-1.2927 0 0.1024" rpy="0 0 0"/>
         <axis xyz="0 1 0"/>
         <limit lower="${radians(-30)}" upper="${radians(30)}" velocity="${infty}" effort="${infty}"/>

Commit message: correct link origins to account for joint origins

File: bmb_description/urdf/aris.urdf.xacro (robot description, xacro)
@@ -33,5 +33,5 @@
             </geometry>
         </visual>
-        <origin xyz="0 0 0" rpy="0 0 0"/>
+        <origin xyz="-0.4244 0 -0.1638" rpy="0 0 0"/>
     </link>
     <joint name="body_to_propeller" type="continuous">
@@ -50,5 +50,5 @@
             </geometry>
         </visual>
-        <origin xyz="-1.45 3.7 1.5" rpy="0.05 0 -0.12"/>
+        <origin xyz="${-1.45 + 0.2649} 3.7 ${1.5 - 0.1714}" rpy="0.05 0 -0.12"/>
     </link>
     <joint name="body_to_left_aileron" type="revolute">
@@ -67,5 +67,5 @@
             </geometry>
         </visual>
-        <origin xyz="-1.45 -3.7 1.5 " rpy="-0.05 0 0.12"/>
+        <origin xyz="${-1.45 + 0.2649} -3.7 ${1.5 - 0.1714}" rpy="-0.05 0 0.12"/>
     </link>
     <joint name="body_to_right_aileron" type="revolute">
@@ -84,5 +84,5 @@
             </geometry>
         </visual>
-        <origin xyz="-5.55 0 0.57" rpy="0 0 0"/>
+        <origin xyz="${-5.55 + 1.2927} 0 ${0.57 - 0.1024}" rpy="0 0 0"/>
     </link>
     <joint name="body_to_elevator" type="revolute">

Commit message: add tiny inertias to all links so Gazebo picks them up

File: bmb_description/urdf/aris.urdf.xacro (robot description, xacro)
@@ -2,4 +2,12 @@
 <robot xmlns:xacro="http://www.ros.org/wiki/xacro" name="aris">
     <xacro:property name="infty" value="${1e9}"/>
+    <xacro:property name="epsilon" value="${1e-9}"/>
+    <xacro:macro name="tiny_inertia">
+        <inertial>
+            <mass value="${epsilon}"/>
+            <inertia ixx="${epsilon}" ixy="0" ixz="0"
+                     iyy="${epsilon}" iyz="0" izz="${epsilon}"/>
+        </inertial>
+    </xacro:macro>
     <link name="body">
         <visual>
@@ -27,4 +35,5 @@
     <!-- Propeller -->
     <link name="propeller">
+        <xacro:tiny_inertia/>
         <visual>
             <geometry>
@@ -44,4 +53,5 @@
     <!-- TODO: use xacro macro for left and right aileron -->
     <link name="left_aileron">
+        <xacro:tiny_inertia/>
         <visual>
             <geometry>
@@ -61,4 +71,5 @@
     <!-- Right Aileron -->
     <link name="right_aileron">
+        <xacro:tiny_inertia/>
         <visual>
             <geometry>
@@ -78,4 +89,5 @@
     <!-- Elevator -->
     <link name="elevator">
+        <xacro:tiny_inertia/>
         <visual>
             <geometry>

Commit message: add tiny collision boxes

File: bmb_description/urdf/aris.urdf.xacro (robot description, xacro)
@@ -3,5 +3,5 @@
     <xacro:property name="infty" value="${1e9}"/>
     <xacro:property name="epsilon" value="${1e-9}"/>
-    <xacro:macro name="tiny_inertia">
+    <xacro:macro name="tiny_inertia_collision">
         <inertial>
             <mass value="${epsilon}"/>
@@ -9,4 +9,9 @@
                      iyy="${epsilon}" iyz="0" izz="${epsilon}"/>
         </inertial>
+        <collision>
+            <geometry>
+                <box size="${epsilon} ${epsilon} ${epsilon}"/>
+            </geometry>
+        </collision>
     </xacro:macro>
     <link name="body">
@@ -35,5 +40,5 @@
     <!-- Propeller -->
     <link name="propeller">
-        <xacro:tiny_inertia/>
+        <xacro:tiny_inertia_collision/>
         <visual>
             <geometry>
@@ -53,5 +58,5 @@
     <!-- TODO: use xacro macro for left and right aileron -->
     <link name="left_aileron">
-        <xacro:tiny_inertia/>
+        <xacro:tiny_inertia_collision/>
         <visual>
             <geometry>
@@ -71,5 +76,5 @@
     <!-- Right Aileron -->
     <link name="right_aileron">
-        <xacro:tiny_inertia/>
+        <xacro:tiny_inertia_collision/>
         <visual>
             <geometry>
@@ -89,5 +94,5 @@
     <!-- Elevator -->
     <link name="elevator">
-        <xacro:tiny_inertia/>
+        <xacro:tiny_inertia_collision/>
         <visual>
             <geometry>

Commit message: rename body to base_link

File: bmb_description/urdf/aris.urdf.xacro (robot description, xacro)
@@ -15,5 +15,5 @@
         </collision>
     </xacro:macro>
-    <link name="body">
+    <link name="base_link">
         <visual>
             <geometry>
@@ -50,5 +50,5 @@
     </link>
     <joint name="body_to_propeller" type="continuous">
-        <parent link="body"/>
+        <parent link="base_link"/>
         <child link="propeller"/>
         <origin xyz="0.4244 0 0.1638" rpy="0 0 0"/>
@@ -68,5 +68,5 @@
     </link>
     <joint name="body_to_left_aileron" type="revolute">
-        <parent link="body"/>
+        <parent link="base_link"/>
         <child link="left_aileron"/>
         <origin xyz="-0.2649 0 0.1714" rpy="0 0 0"/>
@@ -86,5 +86,5 @@
     </link>
     <joint name="body_to_right_aileron" type="revolute">
-        <parent link="body"/>
+        <parent link="base_link"/>
         <child link="right_aileron"/>
         <origin xyz="-0.2649 0 0.1714" rpy="0 0 0"/>
@@ -104,5 +104,5 @@
     </link>
     <joint name="body_to_elevator" type="revolute">
-        <parent link="body"/>
+        <parent link="base_link"/>
         <child link="elevator"/>
         <origin xyz="-1.2927 0 0.1024" rpy="0 0 0"/>
@@ -112,5 +112,5 @@
     <gazebo>
         <plugin name="aris_control" filename="libaris_control_plugin.so">
-            <base_link>body</base_link>
+            <base_link>base_link</base_link>
             <propeller>body_to_propeller</propeller>
             <left_aileron>body_to_left_aileron</left_aileron>

Commit message: increase epsilon. WHY THE FUCK DOES GAZEBO CARE ABOUT THIS!!!!???!?!?

File: bmb_description/urdf/aris.urdf.xacro (robot description, xacro)
@@ -2,5 +2,6 @@
 <robot xmlns:xacro="http://www.ros.org/wiki/xacro" name="aris">
     <xacro:property name="infty" value="${1e9}"/>
-    <xacro:property name="epsilon" value="${1e-9}"/>
+    <!-- Needs to be large enough so Gazebo doesn't ignore the links/joints -->
+    <xacro:property name="epsilon" value="${1e-3}"/>
     <xacro:macro name="tiny_inertia_collision">
         <inertial>

Commit message: update aircraft mass based on actual measurements

File: bmb_description/urdf/aris.urdf.xacro (robot description, xacro)
@@ -29,5 +29,5 @@
         </visual>
         <inertial>
-            <mass value="3.068"/>
+            <mass value="3.3"/>
             <inertia ixx="12.327" ixy="-3.07" ixz="0.739"
                      iyy="1.711" iyz="-2.789" izz="12.659"/>

Commit message: use xacro macro to combine aileron definitions

File: bmb_description/urdf/aris.urdf.xacro (robot description, xacro)
@@ -19,4 +19,26 @@
             <gravity>0</gravity>
         </gazebo>
+    </xacro:macro>
+    <xacro:macro name="aileron" params="prefix">
+        <!-- prefix parameter should be either "left" or "right" -->
+        <xacro:property name="reflect" value="${prefix == 'right' ? 1 : -1}"/>
+        <link name="${prefix}_aileron">
+            <xacro:tiny_inertia_collision/>
+            <visual>
+                <geometry>
+                    <mesh filename="package://bmb_description/meshes/${prefix}_aileron.stl"
+                          scale="0.001 0.001 0.001"/>
+                </geometry>
+            </visual>
+            <origin xyz="-1.45 ${-3.7 * reflect} 1.5"
+                    rpy="${-0.05 * reflect} 0 ${0.12 * reflect}"/>
+        </link>
+        <joint name="body_to_${prefix}_aileron" type="revolute">
+            <parent link="base_link"/>
+            <child link="${prefix}_aileron"/>
+            <origin xyz="-0.2649 0 0.1714" rpy="0 0 0"/>
+            <axis xyz="0 1 0"/>
+            <limit lower="${radians(-30)}" upper="${radians(30)}" velocity="${infty}" effort="${infty}"/>
+        </joint>
     </xacro:macro>
     <link name="base_link">
@@ -60,41 +82,7 @@
         <axis xyz="1 0 0"/>
     </joint>
-    <!-- Left Aileron -->
-    <!-- TODO: use xacro macro for left and right aileron -->
-    <link name="left_aileron">
-        <xacro:tiny_inertia_collision/>
-        <visual>
-            <geometry>
-                <mesh filename="package://bmb_description/meshes/left_aileron.stl"
-                      scale="0.001 0.001 0.001"/>
-            </geometry>
-        </visual>
-        <origin xyz="${-1.45 + 0.2649} 3.7 ${1.5 - 0.1714}" rpy="0.05 0 -0.12"/>
-    </link>
-    <joint name="body_to_left_aileron" type="revolute">
-        <parent link="base_link"/>
-        <child link="left_aileron"/>
-        <origin xyz="-0.2649 0 0.1714" rpy="0 0 0"/>
-        <axis xyz="0 1 0"/>
-        <limit lower="${radians(-30)}" upper="${radians(30)}" velocity="${infty}" effort="${infty}"/>
-    </joint>
-    <!-- Right Aileron -->
-    <link name="right_aileron">
-        <xacro:tiny_inertia_collision/>
-        <visual>
-            <geometry>
-                <mesh filename="package://bmb_description/meshes/right_aileron.stl"
-                      scale="0.001 0.001 0.001"/>
-            </geometry>
-        </visual>
-        <origin xyz="${-1.45 + 0.2649} -3.7 ${1.5 - 0.1714}" rpy="-0.05 0 0.12"/>
-    </link>
-    <joint name="body_to_right_aileron" type="revolute">
-        <parent link="base_link"/>
-        <child link="right_aileron"/>
-        <origin xyz="-0.2649 0 0.1714" rpy="0 0 0"/>
-        <axis xyz="0 1 0"/>
-        <limit lower="${radians(-30)}" upper="${radians(30)}" velocity="${infty}" effort="${infty}"/>
-    </joint>
+    <!-- Ailerons -->
+    <xacro:aileron prefix="right"/>
+    <xacro:aileron prefix="left"/>
     <!-- Elevator -->
     <link name="elevator">

Commit message: take reflect as a parameter

File: bmb_description/urdf/aris.urdf.xacro (robot description, xacro)
@@ -20,7 +20,6 @@
         </gazebo>
     </xacro:macro>
-    <xacro:macro name="aileron" params="prefix">
-        <!-- prefix parameter should be either "left" or "right" -->
-        <xacro:property name="reflect" value="${prefix == 'right' ? 1 : -1}"/>
+    <xacro:macro name="aileron" params="prefix reflect">
+        <!-- TODO: compute reflect based on prefix -->
         <link name="${prefix}_aileron">
             <xacro:tiny_inertia_collision/>
@@ -83,6 +82,6 @@
     </joint>
     <!-- Ailerons -->
-    <xacro:aileron prefix="right"/>
-    <xacro:aileron prefix="left"/>
+    <xacro:aileron prefix="right" reflect="1"/>
+    <xacro:aileron prefix="left" reflect="-1"/>
     <!-- Elevator -->
     <link name="elevator">

Commit message: fixed origins

File: bmb_description/urdf/aris.urdf.xacro (robot description, xacro)
@@ -29,7 +29,6 @@
                           scale="0.001 0.001 0.001"/>
                 </geometry>
+            <origin xyz="0.2649 0 -0.1714" rpy="0 0 0"/>
             </visual>
-            <origin xyz="-1.45 ${-3.7 * reflect} 1.5"
-                    rpy="${-0.05 * reflect} 0 ${0.12 * reflect}"/>
         </link>
         <joint name="body_to_${prefix}_aileron" type="revolute">
@@ -72,6 +71,6 @@
                       scale="0.001 0.001 0.001"/>
             </geometry>
+        <origin xyz="-0.4244 0 -0.1638" rpy="0 0 0"/>
         </visual>
-        <origin xyz="-0.4244 0 -0.1638" rpy="0 0 0"/>
     </link>
     <joint name="body_to_propeller" type="continuous">
@@ -92,6 +91,6 @@
                       scale="0.001 0.001 0.001"/>
             </geometry>
+            <origin xyz="1.2927 0 -0.1024" rpy="0 0 0"/>
         </visual>
-        <origin xyz="${-5.55 + 1.2927} 0 ${0.57 - 0.1024}" rpy="0 0 0"/>
     </link>
     <joint name="body_to_elevator" type="revolute">

Commit message: add dummy link as root, rename base_link to body

File: bmb_description/urdf/aris.urdf.xacro (robot description, xacro)
@@ -29,9 +29,9 @@
                           scale="0.001 0.001 0.001"/>
                 </geometry>
-            <origin xyz="0.2649 0 -0.1714" rpy="0 0 0"/>
+                <origin xyz="0.2649 0 -0.1714" rpy="0 0 0"/>
             </visual>
         </link>
         <joint name="body_to_${prefix}_aileron" type="revolute">
-            <parent link="base_link"/>
+            <parent link="body"/>
             <child link="${prefix}_aileron"/>
             <origin xyz="-0.2649 0 0.1714" rpy="0 0 0"/>
@@ -40,5 +40,7 @@
         </joint>
     </xacro:macro>
-    <link name="base_link">
+    <!-- Need to have a dummy link as the root since the root link should not have an inertia -->
+    <link name="dummy"/>
+    <link name="body">
         <visual>
             <geometry>
@@ -63,4 +65,8 @@
         </gazebo>
     </link>
+    <joint name="dummy_joint" type="fixed">
+        <parent link="dummy"/>
+        <child link="body"/>
+    </joint>
     <!-- Propeller -->
     <link name="propeller">
@@ -71,9 +77,9 @@
                       scale="0.001 0.001 0.001"/>
             </geometry>
-        <origin xyz="-0.4244 0 -0.1638" rpy="0 0 0"/>
+            <origin xyz="-0.4244 0 -0.1638" rpy="0 0 0"/>
         </visual>
     </link>
     <joint name="body_to_propeller" type="continuous">
-        <parent link="base_link"/>
+        <parent link="body"/>
         <child link="propeller"/>
         <origin xyz="0.4244 0 0.1638" rpy="0 0 0"/>
@@ -95,5 +101,5 @@
     </link>
     <joint name="body_to_elevator" type="revolute">
-        <parent link="base_link"/>
+        <parent link="body"/>
         <child link="elevator"/>
         <origin xyz="-1.2927 0 0.1024" rpy="0 0 0"/>
@@ -103,5 +109,5 @@
     <gazebo>
         <plugin name="aris_control" filename="libaris_control_plugin.so">
-            <base_link>base_link</base_link>
+            <base_link>body</base_link>
             <propeller>body_to_propeller</propeller>
             <left_aileron>body_to_left_aileron</left_aileron>

Commit message: correct collision box geometry

File: bmb_description/urdf/aris.urdf.xacro (robot description, xacro)
@@ -57,6 +57,7 @@
         <collision>
             <geometry>
-                <box size="1.5 2.1 0.4"/>
+                <box size="1.6 2.1 0.4"/>
             </geometry>
+            <origin xyz="-0.65 0 0.15" rpy="0 0 0"/>
         </collision>
         <gazebo>

Commit message: remove dummy link since it needs an inertia element for stuff to show up properly in gazebo. I guess we'll just leave the base link with an inertia

File: bmb_description/urdf/aris.urdf.xacro (robot description, xacro)
@@ -40,6 +40,4 @@
         </joint>
     </xacro:macro>
-    <!-- Need to have a dummy link as the root since the root link should not have an inertia -->
-    <link name="dummy"/>
     <link name="body">
         <visual>
@@ -66,8 +64,4 @@
         </gazebo>
     </link>
-    <joint name="dummy_joint" type="fixed">
-        <parent link="dummy"/>
-        <child link="body"/>
-    </joint>
     <!-- Propeller -->
     <link name="propeller">
