Commit message: add link references to gazebo tags

File: bmb_description/urdf/aris.urdf.xacro (robot description, xacro)
@@ -4,5 +4,5 @@
     <!-- Needs to be large enough so Gazebo doesn't ignore the links/joints -->
     <xacro:property name="epsilon" value="${1e-3}"/>
-    <xacro:macro name="tiny_inertia_collision">
+    <xacro:macro name="tiny_inertia_collision" params="link_name">
         <inertial>
             <mass value="${epsilon}"/>
@@ -15,5 +15,5 @@
             </geometry>
         </collision>
-        <gazebo>
+        <gazebo reference="${link_name}">
             <!-- Turn off gravity since the aris_control plugin will apply it -->
             <gravity>0</gravity>
@@ -23,5 +23,5 @@
         <!-- TODO: compute reflect based on prefix -->
         <link name="${prefix}_aileron">
-            <xacro:tiny_inertia_collision/>
+            <xacro:tiny_inertia_collision link_name="${prefix}_aileron"/>
             <visual>
                 <geometry>
@@ -59,5 +59,5 @@
             <origin xyz="-0.65 0 0.15" rpy="0 0 0"/>
         </collision>
-        <gazebo>
+        <gazebo reference="body">
             <!-- Turn off gravity since the aris_control plugin will apply it -->
             <gravity>0</gravity>
@@ -66,5 +66,5 @@
     <!-- Propeller -->
     <link name="propeller">
-        <xacro:tiny_inertia_collision/>
+        <xacro:tiny_inertia_collision link_name="propeller"/>
         <visual>
             <geometry>
@@ -86,5 +86,5 @@
     <!-- Elevator -->
     <link name="elevator">
-        <xacro:tiny_inertia_collision/>
+        <xacro:tiny_inertia_collision link_name="elevator"/>
         <visual>
             <geometry>

Commit message: move gazebo tags outside of links

File: bmb_description/urdf/aris.urdf.xacro (robot description, xacro)
@@ -4,5 +4,5 @@
     <!-- Needs to be large enough so Gazebo doesn't ignore the links/joints -->
     <xacro:property name="epsilon" value="${1e-3}"/>
-    <xacro:macro name="tiny_inertia_collision" params="link_name">
+    <xacro:macro name="tiny_inertia_collision">
         <inertial>
             <mass value="${epsilon}"/>
@@ -15,13 +15,9 @@
             </geometry>
         </collision>
-        <gazebo reference="${link_name}">
-            <!-- Turn off gravity since the aris_control plugin will apply it -->
-            <gravity>0</gravity>
-        </gazebo>
     </xacro:macro>
     <xacro:macro name="aileron" params="prefix reflect">
         <!-- TODO: compute reflect based on prefix -->
         <link name="${prefix}_aileron">
-            <xacro:tiny_inertia_collision link_name="${prefix}_aileron"/>
+            <xacro:tiny_inertia_collision/>
             <visual>
                 <geometry>
@@ -59,12 +55,8 @@
             <origin xyz="-0.65 0 0.15" rpy="0 0 0"/>
         </collision>
-        <gazebo reference="body">
-            <!-- Turn off gravity since the aris_control plugin will apply it -->
-            <gravity>0</gravity>
-        </gazebo>
     </link>
     <!-- Propeller -->
     <link name="propeller">
-        <xacro:tiny_inertia_collision link_name="propeller"/>
+        <xacro:tiny_inertia_collision/>
         <visual>
             <geometry>
@@ -86,5 +78,5 @@
     <!-- Elevator -->
     <link name="elevator">
-        <xacro:tiny_inertia_collision link_name="elevator"/>
+        <xacro:tiny_inertia_collision/>
         <visual>
             <geometry>
@@ -102,4 +94,17 @@
         <limit lower="${radians(-30)}" upper="${radians(30)}" velocity="${infty}" effort="${infty}"/>
     </joint>
+    <!-- Turn off gravity for each link since the aris_control plugin will apply it -->
+    <gazebo reference="body">
+        <gravity>0</gravity>
+    </gazebo>
+    <gazebo reference="right_aileron">
+        <gravity>0</gravity>
+    </gazebo>
+    <gazebo reference="left_aileron">
+        <gravity>0</gravity>
+    </gazebo>
+    <gazebo reference="elevator">
+        <gravity>0</gravity>
+    </gazebo>
     <gazebo>
         <plugin name="aris_control" filename="libaris_control_plugin.so">

Commit message: add color to model

File: bmb_description/urdf/aris.urdf.xacro (robot description, xacro)
@@ -16,4 +16,13 @@
         </collision>
     </xacro:macro>
+    <material name="black">
+        <color rgba="0 0 0 0.8"/>
+    </material>
+    <material name="gold">
+        <color rgba="0.7 0.6 0.4 0.9"/>
+    </material>
+    <material name="green">
+        <color rgba="0.3 0.9 0.2 1"/>
+    </material>
     <xacro:macro name="aileron" params="prefix reflect">
         <!-- TODO: compute reflect based on prefix -->
@@ -26,4 +35,5 @@
                 </geometry>
                 <origin xyz="0.2649 0 -0.1714" rpy="0 0 0"/>
+                <material name="gold"/>
             </visual>
         </link>
@@ -43,4 +53,5 @@
                       scale="0.001 0.001 0.001"/>
             </geometry>
+            <material name="black"/>
         </visual>
         <inertial>
@@ -65,4 +76,5 @@
             </geometry>
             <origin xyz="-0.4244 0 -0.1638" rpy="0 0 0"/>
+            <material name="green"/>
         </visual>
     </link>
@@ -85,4 +97,5 @@
             </geometry>
             <origin xyz="1.2927 0 -0.1024" rpy="0 0 0"/>
+            <material name="gold"/>
         </visual>
     </link>
